File: KiCAD/PSU-Plus.kicad_pcb (KiCad board)
At the start: 2 copper layers, 18 x 49.5 mm, 55 parts, among them U1 AP62301Z6-7, U2 AP62301Z6-7, U3 AP62301Z6-7, U4 AP62301Z6-7, U5 AP62301Z6-7

Commit message: Schematic refreshing, redoing PCB layout, gerbers
Parts:
- added REF**: OSHW-Logo2_7.3x6mm_SilkScreen, Symbol:OSHW-Logo2_7.3x6mm_SilkScreen, B.Cu at (173.9, 144.6)
- L1, L2, L3, L4, L5: footprint PSU Plus:1919 -> Inductor_SMD:L_Chilisin_BMRx00050512-B
- U1, U2, U3, U4, U5: value AP62301Z6-7 -> AP62301Z6; footprint PSU Plus:SOT-563mod -> Package_TO_SOT_SMD:SOT-563
- moved C13 0.45 mm to (170.4, 113.5)
- moved C17 0.45 mm to (170.4, 105.5)
- moved C1 0.45 mm to (170.4, 137.5)
- moved C5 0.40 mm to (170.4, 129.6)
- moved C9 0.40 mm to (170.4, 121.6)
- moved C11 0.10 mm to (174.4, 126.8)
- moved C15 0.10 mm to (174.4, 118.7)
- moved C19 0.10 mm to (174.4, 110.7)
- moved C3 0.10 mm to (174.4, 142.7)
- moved C7 0.10 mm to (174.4, 134.8)
- renumbered VIN to TP1, GND to TP10, 5V to TP11, GND to TP12, VIN to TP13, 1V to TP2, GND to TP3, GND to TP4, 1V15 to TP5, GND to TP6, 1V8 to TP7, GND to TP8, 3V3 to TP9
Connections:
- net Net-(C11-Pad1) renamed +1V8
- net Net-(C15-Pad1) renamed +3V3
- net Net-(C19-Pad1) renamed +5V
- net Net-(C3-Pad1) renamed +1V0
- net Net-(C7-Pad1) renamed +1V15
- net VIN renamed VBUS
Other:
- board text added: "bitbuilt.net"
