File: KiCAD/PSU-Plus.kicad_sch (KiCad schematic)
At the start: 55 parts, among them U1 AP62301Z6-7, U2 AP62301Z6-7, U3 AP62301Z6-7, U4 AP62301Z6-7, U5 AP62301Z6-7

Commit message: Schematic refreshing, redoing PCB layout, gerbers
Parts:
- removed U1, U2, U3, U4, U5: AP62301Z6-7, PSU Plus:SOT-563mod, symbol PSU:AP62301Z6-7
- added U1, U2, U3, U4, U5: AP62301Z6, Package_TO_SOT_SMD:SOT-563, symbol Regulator_Switching:AP62300Z6
- C1, C13, C17, C5, C9: symbol Device:C -> Device:C_Small
- L1, L2, L3, L4, L5: footprint PSU Plus:1919 -> Inductor_SMD:L_Chilisin_BMRx00050512-B
Connections:
- net GND: now also U1.3 (GND), U2.3 (GND), U3.3 (GND), U4.3 (GND), U5.3 (GND)
- net at C1.2, L1.1: now also U1.2 (SW)
- net at C1.1: now also U1.4 (BST)
- net at R1.2, R2.1: now also U1.6 (FB)
- net +1V0: now reaches C3.1, C4.1, L1.2, R1.1, TP2.1
- net at C5.2, L2.1: now also U2.2 (SW)
- net at C5.1: now also U2.4 (BST)
- net at R3.2, R4.1: now also U2.6 (FB)
- net +1V15: now reaches C7.1, C8.1, L2.2, R3.1, TP5.1
- net at C10.2, JP1.2 (B): now also U3.1 (VIN)
- net at C9.2, L3.1: now also U3.2 (SW)
- net at C9.1: now also U3.4 (BST)
- net at R5.2, R6.1: now also U3.6 (FB)
- net +1V8: now reaches C11.1, C12.1, L3.2, R5.1, TP7.1
- net at C13.2, L4.1: now also U4.2 (SW)
- net at C13.1: now also U4.4 (BST)
- net at R7.2, R8.1: now also U4.6 (FB)
- net +3V3: now reaches C15.1, C16.1, L4.2, R7.1, TP9.1
- net at C18.2, JP2.2 (B): now also U5.1 (VIN)
- net at C17.2, L5.1: now also U5.2 (SW)
- net at C17.1: now also U5.4 (BST)
- net at R10.1, R9.2: now also U5.6 (FB)
- net +5V: now reaches C19.1, C20.1, L5.2, R9.1, TP11.1
- net VIN renamed VBUS
- net VBUS: now also U1.1 (VIN), U2.1 (VIN), U4.1 (VIN)
Other:
- moved on the sheet: C1, C10, C13, C14, C17, C18, C5, C9, JP1, L1
